Commit message: fix bug x1 is not added always

File: urdf/rrbot.xacro (robot description, xacro)
@@ -86,5 +86,5 @@
       <origin xyz="0 0 0.5" rpy="0 0 0"/>
       <geometry>
-	<box size="0.00 0.00 0.95"/>
+	<box size="0.00001 0.00001 0.95"/>
       </geometry>
       <color rgba="0 0 0 0"/>

Commit message: applied a weird trick for quaternion (in CLC.cpp line 290)

File: urdf/rrbot.xacro (robot description, xacro)
@@ -20,4 +20,5 @@
     <child link="rect"/>
     <origin xyz="0.15 0.45 0.00000" rpy="0 0 -0.61546"/>
+    <!--<origin xyz="0.0 0.0 0.00000" rpy="0 0 -0.61546"/>-->
     <axis xyz="0 0 1"/>
   </joint>
